File: register_general.kicad_pcb (KiCad board)
At the start: 4 copper layers, 76 x 28 mm, 29 parts, among them J1 Conn_01x16_Pin, J2 Conn_01x16_Pin, J3 load select, J4 output select, U1 74HC245, U2 74HC377

Commit message: Add vias, GND planes, QR code, version and other details
Parts:
- moved C2 4.11 mm to (114.8, 87.5), turned to -90 degrees
- moved C3 2.68 mm to (122.9, 81.0)
- moved D10 0.60 mm to (138.2, 67.3)
- moved R10 0.60 mm to (134.4, 67.3)
Routing:
- net +5V: track 146.8 -> 148.9 mm
- net reg2_out: track 64.7 -> 63.6 mm
- net Net-(J4-Pin_2): track 63.6 -> 62.9 mm
- net /dbus7: track 70.8 -> 70.1 mm
- net /q6: track 38.5 -> 37.8 mm
- net /q3: track 47.4 -> 46.8 mm
- net GND: vias 57 -> 106
Other:
- board text added: "Rev 1.0 2026/03"
