File: CAD/register_general/register_general.kicad_pcb (KiCad board)
At the start: 2 copper layers, 75 x 28 mm, 42 parts, among them J1 Conn_01x16_Pin, J2 Conn_01x16_Pin, U1 74HC245, U2 74HC377

Commit message: layout changes
Parts:
- moved FID2 15.1 mm to (145.0, 90.1)
- moved FID1 6.65 mm to (85.0, 66.5)
- moved D10 0.36 mm to (134.5, 71.1)
- moved R10 0.36 mm to (133.6, 68.0)
- moved C3 0.11 mm to (88.9, 67.3)
Routing:
- net /q4: track 32.6 -> 33.5 mm
- net ~{reg1_in}: track 28.6 -> 29.4 mm
- net ~{reg1_out}: track 66.9 -> 67.2 mm, vias 2 -> 4
- net GND: vias 62 -> 71
