File: CAD/program_counter/program_counter.kicad_pcb (KiCad board)
At the start: 2 copper layers, 100 x 50 mm, 59 parts, among them J1 Conn_01x18_Pin, J2 Conn_01x06_Pin, SW1 SW_Push, SW2 SW_Push, U1 74HC161, U2 74HC161, U3 74HC161, U4 74HC161, U5 74HC245, U6 74HC245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

Commit message: PC layout changes
Parts:
- moved FID2 13.0 mm to (134.5, 59.2)
- moved TP1 0.60 mm to (137.0, 87.8)
- moved TP2 0.60 mm to (137.0, 93.8)
- moved TP3 0.50 mm to (98.1, 87.3)
- moved TP4 0.50 mm to (98.1, 93.3)
Routing:
- net +5V: track 397.7 -> 400.0 mm
- net /xtal1: track 10.6 -> 11.8 mm
- net ~{RESET}: track 172.9 -> 173.8 mm
- net ~{pc_H_in}: track 86.5 -> 87.1 mm
- net GND: vias 137 -> 153
