File: CAD/control_logic_unit/control_logic_unit.kicad_pcb (KiCad board)
At the start: 2 copper layers, 0 parts

Commit message: finish CLU schematic and PCB
Parts:
- added C1: 100nF, Capacitor_SMD:C_0805_2012Metric, F.Cu at (59.0, 40.5)
- added C10: 10uF, Capacitor_SMD:C_0805_2012Metric, F.Cu at (138.2, 30.7)
- added C2: 100nF, Capacitor_SMD:C_0805_2012Metric, F.Cu at (87.6, 40.5)
- added C3: 100nF, Capacitor_SMD:C_0805_2012Metric, F.Cu at (116.2, 40.5)
- added C4: 100nF, Capacitor_SMD:C_0805_2012Metric, F.Cu at (55.5, 69.6)
- added C5: 100nF, Capacitor_SMD:C_0805_2012Metric, F.Cu at (69.7, 69.6)
- added C6: 100nF, Capacitor_SMD:C_0805_2012Metric, F.Cu at (84.0, 69.6)
- added C7: 100nF, Capacitor_SMD:C_0805_2012Metric, F.Cu at (98.2, 69.6)
- added C8: 100nF, Capacitor_SMD:C_0805_2012Metric, F.Cu at (112.7, 69.6)
- added C9: 100nF, Capacitor_SMD:C_0805_2012Metric, F.Cu at (126.8, 69.6)
- added FID1: Fiducial, Fiducial:Fiducial_0.5mm_Mask1mm, F.Cu at (127.5, 37.7)
- added FID2: Fiducial, Fiducial:Fiducial_0.5mm_Mask1mm, F.Cu at (60.2, 70.1)
- added H1: MountingHole_Pad, MountingHole:MountingHole_2.5mm_Pad_Via, F.Cu at (45.4, 94.5)
- added H2: MountingHole_Pad, MountingHole:MountingHole_2.5mm_Pad_Via, F.Cu at (45.4, 37.5)
- added H3: ToolingHole, MountingHole:ToolingHole_1.152mm, F.Cu at (140.9, 96.0)
- added H4: ToolingHole, MountingHole:ToolingHole_1.152mm, F.Cu at (140.9, 29.0)
- added H5: ToolingHole, MountingHole:ToolingHole_1.152mm, F.Cu at (43.9, 90.5)
- added H6: ToolingHole, MountingHole:ToolingHole_1.152mm, F.Cu at (43.9, 41.5)
- added J1: Conn_01x18_Pin, Connector_PinHeader_2.54mm:PinHeader_2x23_P2.54mm_Horizontal, F.Cu at (137.2, 34.5)
- added J2: Conn_01x28_Pin, Connector_PinSocket_2.54mm:PinSocket_1x28_P2.54mm_Vertical, F.Cu at (55.6, 93.5)
- added J3: Conn_01x02_Pin, Connector_PinSocket_2.54mm:PinSocket_1x02_P2.54mm_Vertical, F.Cu at (46.4, 31.5)
- added J4: Conn_01x02_Pin, Connector_PinSocket_2.54mm:PinSocket_1x02_P2.54mm_Vertical, F.Cu at (130.4, 31.5)
- added R1: 10k, Resistor_SMD:R_0805_2012Metric, F.Cu at (119.1, 88.5)
- added RN1: 10k, Resistor_SMD:R_Array_Convex_4x0603, F.Cu at (61.9, 88.5)
- added RN2: 10k, Resistor_SMD:R_Array_Convex_4x0603, F.Cu at (72.1, 88.5)
- added RN3: 10k, Resistor_SMD:R_Array_Convex_4x0603, F.Cu at (82.3, 88.5)
- added RN4: 10k, Resistor_SMD:R_Array_Convex_4x0603, F.Cu at (92.5, 88.5)
- added RN5: 10k, Resistor_SMD:R_Array_Convex_4x0603, F.Cu at (102.6, 88.5)
- added RN6: 10k, Resistor_SMD:R_Array_Convex_4x0603, F.Cu at (112.8, 88.5)
- added Ref**: Val**, 8-bit_computer:by-nc-sa.eu, B.Cu at (124.9, 69.9)
- added TP1: TestPoint, TestPoint:TestPoint_THTPad_D1.0mm_Drill0.5mm, F.Cu at (47.1, 85.5)
- added TP2: TestPoint, TestPoint:TestPoint_THTPad_D1.0mm_Drill0.5mm, F.Cu at (51.2, 89.8)
- added U1: SST39SF010, 8-bit_computer:PLCC-32_THT-Socket, F.Cu at (60.3, 48.6)
- added U2: SST39SF010, 8-bit_computer:PLCC-32_THT-Socket, F.Cu at (88.9, 48.6)
- added U3: SST39SF010, 8-bit_computer:PLCC-32_THT-Socket, F.Cu at (117.5, 48.6)
- added U4: 74HC157, Package_SO:SO-16_3.9x9.9mm_P1.27mm, F.Cu at (51.9, 77.1)
- added U5: 74HC157, Package_SO:SO-16_3.9x9.9mm_P1.27mm, F.Cu at (66.1, 77.1)
- added U6: 74HC157, Package_SO:SO-16_3.9x9.9mm_P1.27mm, F.Cu at (80.5, 77.1)
- added U7: 74HC157, Package_SO:SO-16_3.9x9.9mm_P1.27mm, F.Cu at (94.7, 77.1)
- added U8: 74HC157, Package_SO:SO-16_3.9x9.9mm_P1.27mm, F.Cu at (109.1, 77.1)
- added U9: 74HC157, Package_SO:SO-16_3.9x9.9mm_P1.27mm, F.Cu at (123.3, 77.1)
Routing:
- net +5V: track 0.00 -> 427.2 mm, vias 0 -> 6
- net man_ctrl: track 0.00 -> 163.0 mm, vias 0 -> 7
- net /opcode.0: track 0.00 -> 157.7 mm, vias 0 -> 3
- net /opcode.1: track 0.00 -> 157.0 mm, vias 0 -> 3
- net /opcode.3: track 0.00 -> 145.5 mm, vias 0 -> 3
- net /opcode.2: track 0.00 -> 144.8 mm, vias 0 -> 3
- net /opcode.4: track 0.00 -> 138.5 mm, vias 0 -> 6
- net /opcode.5: track 0.00 -> 133.6 mm, vias 0 -> 3
- net /step.0: track 0.00 -> 129.1 mm, vias 0 -> 3
- net INTERRUPT: track 0.00 -> 128.3 mm, vias 0 -> 3
- net /aflags.zf: track 0.00 -> 125.3 mm, vias 0 -> 6
- net /aflags.vf: track 0.00 -> 122.3 mm, vias 0 -> 3
- net /aflags.cf: track 0.00 -> 121.7 mm, vias 0 -> 3
- net FETCH: track 0.00 -> 117.9 mm, vias 0 -> 3
- net /step.1: track 0.00 -> 116.7 mm, vias 0 -> 3
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- added copper zone on B.Cu, net GND
- added copper zone on F.Cu, net GND
Other:
- board outline added: 100 x 70 mm
- board text added: "5V"
- board text added: "CONTROL LOGIC UNIT"
- board text added: "GND"
- board text added: "Rev ${REVISION} ${YEAR}/${MONTH}"
- board text added: "S/N"
- board text added: "github.com/${GITHUB}"

Commit message: CLU Controls Shield layout changes, add reg2 select switch, CLU layout changes
Parts:
- J2: value Conn_01x28_Pin -> Conn_01x30_Pin; footprint Connector_PinSocket_2.54mm:PinSocket_1x28_P2.54mm_Vertical -> Connector_PinSocket_2.54mm:PinSocket_1x30_P2.54mm_Vertical
- U1, U2, U3: value SST39SF010 -> SST39SF040
- moved C10 9.26 mm to (130.2, 35.5), turned to -90 degrees
- moved R1 5.10 mm to (124.2, 88.5)
- moved RN2 2.60 mm to (69.5, 88.5)
- moved RN3 2.60 mm to (79.7, 88.5)
- moved RN4 2.60 mm to (89.9, 88.5)
- moved RN5 2.60 mm to (100.0, 88.5)
- moved RN6 2.60 mm to (110.2, 88.5)
- moved RN1 2.50 mm to (59.4, 88.5)
- moved J4 2.24 mm to (132.4, 30.5)
- moved J3 1.00 mm to (46.4, 30.5)
Connections:
- J1 pad 10: /opcode.2 -> /opcode.4
- J1 pad 11: /opcode.3 -> /opcode.5
- J1 pad 12: /opcode.4 -> /aflags.zf
- J1 pad 13: /opcode.5 -> /aflags.cf
- J1 pad 14: /aflags.zf -> /aflags.nf
- J1 pad 15: /aflags.cf -> /aflags.vf
- J1 pad 16: /aflags.nf -> /step.0
- J1 pad 17: /aflags.vf -> /step.1
- J1 pad 18: /step.0 -> /step.2
- J1 pad 19: /step.1 -> /step.3
- J1 pad 20: /step.2 -> /q1.0
- J1 pad 21: /step.3 -> /q1.1
- J1 pad 22: /q1.0 -> /q1.2
- J1 pad 23: /q1.1 -> /q1.3
- J1 pad 24: /q1.2 -> /q1.4
- J1 pad 25: /q1.3 -> /q1.5
- J1 pad 26: /q1.4 -> /q1.6
- J1 pad 27: /q1.5 -> /q1.7
- J1 pad 28: /q1.6 -> /q2.0
- J1 pad 29: /q1.7 -> /q2.1
- J1 pad 3: clk -> FETCH
- J1 pad 30: /q2.0 -> /q2.2
- J1 pad 31: /q2.1 -> /q2.3
- J1 pad 32: /q2.2 -> /q2.4
- J1 pad 33: /q2.3 -> /q2.5
- J1 pad 34: /q2.4 -> /q2.6
- J1 pad 35: /q2.5 -> /q2.7
- J1 pad 36: /q2.6 -> /q3.0
- J1 pad 37: /q2.7 -> /q3.1
- J1 pad 38: /q3.0 -> /q3.2
- J1 pad 39: /q3.1 -> /q3.3
- J1 pad 4: ~{rst} -> EXECUTE
- J1 pad 40: /q3.2 -> /q3.4
- J1 pad 41: /q3.3 -> /q3.5
- J1 pad 42: /q3.4 -> /q3.6
- J1 pad 43: /q3.5 -> /q3.7
- J1 pad 44: /q3.6 -> /reg2_sig.0
- J1 pad 45: /q3.7 -> /reg2_sig.1
- J1 pad 46: GND -> /reg2_sig.2
- J1 pad 5: FETCH -> INTERRUPT
- J1 pad 6: EXECUTE -> /opcode.0
- J1 pad 7: INTERRUPT -> /opcode.1
- J1 pad 8: /opcode.0 -> /opcode.2
- J1 pad 9: /opcode.1 -> /opcode.3
- J2 pad 1: GND -> /sig1.0
- J2 pad 10: /sig2.0 -> /sig2.1
- J2 pad 11: /sig2.1 -> /sig2.2
- J2 pad 12: /sig2.2 -> /sig2.3
- J2 pad 13: /sig2.3 -> /sig2.4
- J2 pad 14: /sig2.4 -> /sig2.5
- J2 pad 15: /sig2.5 -> /sig2.6
- J2 pad 16: /sig2.6 -> /sig2.7
- J2 pad 17: /sig2.7 -> /sig3.0
- J2 pad 18: /sig3.0 -> /sig3.1
- J2 pad 19: /sig3.1 -> /sig3.2
- J2 pad 2: /sig1.0 -> /sig1.1
- J2 pad 20: /sig3.2 -> /sig3.3
- J2 pad 21: /sig3.3 -> /sig3.4
- J2 pad 22: /sig3.4 -> /sig3.5
- J2 pad 23: /sig3.5 -> /sig3.6
- J2 pad 24: /sig3.6 -> /sig3.7
- J2 pad 25: /sig3.7 -> /reg2_sig.0
- J2 pad 26: man_ctrl -> /reg2_sig.1
- J2 pad 27: +5V -> /reg2_sig.2
- J2 pad 28: GND -> man_ctrl
- J2 pad 3: /sig1.1 -> /sig1.2
- J2 pad 4: /sig1.2 -> /sig1.3
- J2 pad 5: /sig1.3 -> /sig1.4
- J2 pad 6: /sig1.4 -> /sig1.5
- J2 pad 7: /sig1.5 -> /sig1.6
- J2 pad 8: /sig1.6 -> /sig1.7
- J2 pad 9: /sig1.7 -> /sig2.0
- J4 pad 2: GND -> +5V
- U1 pad 1: unconnected-(U1-NC-Pad1) -> GND
- U1 pad 30: unconnected-(U1-NC-Pad30) -> GND
- U2 pad 1: unconnected-(U2-NC-Pad1) -> GND
- U2 pad 30: unconnected-(U2-NC-Pad30) -> GND
- U3 pad 1: unconnected-(U3-NC-Pad1) -> GND
- U3 pad 30: unconnected-(U3-NC-Pad30) -> GND
Routing:
- net /reg2_sig.0: track 0.00 -> 25.5 mm
- net /reg2_sig.1: track 0.00 -> 19.4 mm
- net /reg2_sig.2: track 0.00 -> 19.4 mm
- net /sig3.7: track 28.6 -> 32.1 mm
- net /aflags.cf: track 121.7 -> 118.3 mm
- net /opcode.5: track 133.6 -> 130.3 mm
- net /aflags.zf: track 125.3 -> 122.0 mm
- net /aflags.vf: track 122.3 -> 119.1 mm
- net /aflags.nf: track 116.6 -> 113.4 mm
- net /opcode.4: track 138.5 -> 135.3 mm
- net /opcode.3: track 145.5 -> 142.5 mm
- net /step.0: track 129.1 -> 126.1 mm
- net /step.1: track 116.7 -> 113.9 mm
- net /opcode.2: track 144.8 -> 142.0 mm
- net /opcode.1: track 157.0 -> 154.3 mm
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