File: CAD/control_logic_unit/control_logic_unit.kicad_sch (KiCad schematic)
At the start: 85 parts, among them J1 Conn_01x18_Pin, SW1 SW_DIP_x08, SW2 SW_DIP_x08, SW3 SW_DIP_x08, SW4 SW_DPDT_x2, U1 SST39SF010, U2 SST39SF010, U3 SST39SF010

Commit message: finish CLU schematic and PCB
Parts:
- removed D1, D10, D11, D12, D13, D14, D15, D16, D17, D18, D19, D2, D20, D21, D22, D23, D24, D3, D4, D5, D6, D7, D8, D9: LED, symbol Device:LED
- removed R10, R11, R12, R13, R14, R15, R16, R17, R18, R19, R2, R20, R21, R22, R23, R24, R25, R3, R4, R5, R6, R7, R8, R9: 10k, symbol Device:R
- removed R26, R27, R28, R29, R30, R31, R32, R33, R34, R35, R36, R37, R38, R39, R40, R41, R42, R43, R44, R45, R46, R47, R48, R49: 1k, symbol Device:R
- removed SW1, SW2, SW3: SW_DIP_x08, symbol Switch:SW_DIP_x08
- removed SW4: SW_DPDT_x2, symbol Switch:SW_DPDT_x2
- added C4, C5, C6, C7, C8, C9: 100nF, Capacitor_SMD:C_0805_2012Metric, symbol Device:C
- added FID1, FID2: Fiducial, Fiducial:Fiducial_0.5mm_Mask1mm, symbol Mechanical:Fiducial
- added H1, H2: MountingHole_Pad, MountingHole:MountingHole_2.5mm_Pad_Via, symbol Mechanical:MountingHole_Pad
- added H3, H4, H5, H6: ToolingHole, MountingHole:ToolingHole_1.152mm, symbol Mechanical:MountingHole
- added J2: Conn_01x28_Pin, Connector_PinSocket_2.54mm:PinSocket_1x28_P2.54mm_Vertical, symbol Connector:Conn_01x28_Pin
- added J3, J4: Conn_01x02_Pin, Connector_PinSocket_2.54mm:PinSocket_1x02_P2.54mm_Vertical, symbol Connector:Conn_01x02_Pin
- added RN1, RN2, RN3, RN4, RN5, RN6: 10k, Resistor_SMD:R_Array_Convex_4x0603, symbol Device:R_Pack04
- added TP1, TP2: TestPoint, TestPoint:TestPoint_THTPad_D1.0mm_Drill0.5mm, symbol Connector:TestPoint
- added U4, U5, U6, U7, U8, U9: 74HC157, Package_SO:SO-16_3.9x9.9mm_P1.27mm, symbol 8bit_computer:74HC157
- C1, C2, C3: footprint (none) -> Capacitor_SMD:C_0805_2012Metric
- J1: footprint Connector_PinHeader_2.54mm:PinHeader_2x09_P2.54mm_Horizontal -> Connector_PinHeader_2.54mm:PinHeader_2x23_P2.54mm_Horizontal
- R1: footprint (none) -> Resistor_SMD:R_0805_2012Metric
- U1, U2, U3: footprint Package_LCC:PLCC-32_THT-Socket -> 8-bit_computer:PLCC-32_THT-Socket
- renumbered C9 to C10
Connections:
- net ~{rom_oe} is gone; now on net GND: U1.22 (CE), U1.24 (OE), U2.22 (CE), U2.24 (OE), U3.22 (CE), U3.24 (OE)
- net +5V: now also C1.2, C2.2, C3.2, C4.1, C5.1, C6.1, C7.1, C8.1, C9.1, J2.27 (Pin_27), TP1.1, U4.16 (VCC), U5.16 (VCC), U6.16 (VCC), U7.16 (VCC), U8.16 (VCC), U9.16 (VCC); no longer C1.1, C2.1, C3.1
- net EXECUTE: now also J1.6 (Pin_6); no longer J1.44 (Pin_44)
- net FETCH: now also J1.5 (Pin_5); no longer J1.43 (Pin_43)
- net GND: now also C1.1, C2.1, C3.1, R1.2, C4.2, C5.2, C6.2, C7.2, C8.2, C9.2, H1.1, H2.1, J2.1 (Pin_1), J2.28 (Pin_28), J3.1 (Pin_1), J3.2 (Pin_2), J4.1 (Pin_1), J4.2 (Pin_2), RN1.5 (R4.2), RN1.6 (R3.2), RN1.7 (R2.2), RN1.8 (R1.2), RN2.5 (R4.2), RN2.6 (R3.2), RN2.7 (R2.2), RN2.8 (R1.2), RN3.5 (R4.2), RN3.6 (R3.2), RN3.7 (R2.2), RN3.8 (R1.2), RN4.5 (R4.2), RN4.6 (R3.2), RN4.7 (R2.2), RN4.8 (R1.2), RN5.5 (R4.2), RN5.6 (R3.2), RN5.7 (R2.2), RN5.8 (R1.2), RN6.5 (R4.2), RN6.6 (R3.2), RN6.7 (R2.2), RN6.8 (R1.2), TP2.1, U4.15 (E), U4.8 (GND), U5.15 (E), U5.8 (GND), U6.15 (E), U6.8 (GND), U7.15 (E), U7.8 (GND), U8.15 (E), U8.8 (GND), U9.15 (E), U9.8 (GND); no longer C1.2, C2.2, C3.2, R1.1
- net INTERRUPT: now also J1.7 (Pin_7); no longer J1.45 (Pin_45)
- net aflags.cf: now also J1.15 (Pin_15); no longer J1.36 (Pin_36)
- net aflags.nf: now also J1.16 (Pin_16); no longer J1.37 (Pin_37)
- net aflags.vf: now also J1.17 (Pin_17); no longer J1.38 (Pin_38)
- net aflags.zf: now also J1.14 (Pin_14); no longer J1.35 (Pin_35)
- net opcode.0: now also J1.8 (Pin_8); no longer J1.29 (Pin_29)
- net opcode.1: now also J1.9 (Pin_9); no longer J1.30 (Pin_30)
- net opcode.2: now also J1.10 (Pin_10); no longer J1.31 (Pin_31)
- net opcode.3: now also J1.11 (Pin_11); no longer J1.32 (Pin_32)
- net opcode.4: now also J1.12 (Pin_12); no longer J1.33 (Pin_33)
- net opcode.5: now also J1.13 (Pin_13); no longer J1.34 (Pin_34)
- net q1.0: now also J1.22 (Pin_22), U4.4 (Za); no longer J1.5 (Pin_5), R1.2, U1.13 (D0)
- net q1.1: now also J1.23 (Pin_23), U4.7 (Zb); no longer J1.6 (Pin_6), U1.14 (D1)
- net q1.2: now also J1.24 (Pin_24), U4.9 (Zc); no longer J1.7 (Pin_7), U1.15 (D2)
- net q1.3: now also J1.25 (Pin_25), U4.12 (Zd); no longer J1.8 (Pin_8), U1.17 (D3)
- net q1.4: now also J1.26 (Pin_26), U5.4 (Za); no longer J1.9 (Pin_9), U1.18 (D4)
- net q1.5: now also J1.27 (Pin_27), U5.7 (Zb); no longer J1.10 (Pin_10), U1.19 (D5)
- net q1.6: now also J1.28 (Pin_28), U5.9 (Zc); no longer J1.11 (Pin_11), U1.20 (D6)
- net q1.7: now also J1.29 (Pin_29), U5.12 (Zd); no longer J1.12 (Pin_12), U1.21 (D7)
- net q2.0: now also J1.30 (Pin_30), U6.4 (Za); no longer J1.13 (Pin_13), U2.13 (D0)
- net q2.1: now also J1.31 (Pin_31), U6.7 (Zb); no longer J1.14 (Pin_14), U2.14 (D1)
- net q2.2: now also J1.32 (Pin_32), U6.9 (Zc); no longer J1.15 (Pin_15), U2.15 (D2)
- net q2.3: now also J1.33 (Pin_33), U6.12 (Zd); no longer J1.16 (Pin_16), U2.17 (D3)
- net q2.4: now also J1.34 (Pin_34), U7.4 (Za); no longer J1.17 (Pin_17), U2.18 (D4)
- net q2.5: now also J1.35 (Pin_35), U7.7 (Zb); no longer J1.18 (Pin_18), U2.19 (D5)
- net q2.6: now also J1.36 (Pin_36), U7.9 (Zc); no longer J1.19 (Pin_19), U2.20 (D6)
- net q2.7: now also J1.37 (Pin_37), U7.12 (Zd); no longer J1.20 (Pin_20), U2.21 (D7)
- net q3.0: now also J1.38 (Pin_38), U8.4 (Za); no longer J1.21 (Pin_21), U3.13 (D0)
- net q3.1: now also J1.39 (Pin_39), U8.7 (Zb); no longer J1.22 (Pin_22), U3.14 (D1)
- net q3.2: now also J1.40 (Pin_40), U8.9 (Zc); no longer J1.23 (Pin_23), U3.15 (D2)
- net q3.3: now also J1.41 (Pin_41), U8.12 (Zd); no longer J1.24 (Pin_24), U3.17 (D3)
- net q3.4: now also J1.42 (Pin_42), U9.4 (Za); no longer J1.25 (Pin_25), U3.18 (D4)
- net q3.5: now also J1.43 (Pin_43), U9.7 (Zb); no longer J1.26 (Pin_26), U3.19 (D5)
- net q3.6: now also J1.44 (Pin_44), U9.9 (Zc); no longer J1.27 (Pin_27), U3.20 (D6)
- net q3.7: now also J1.45 (Pin_45), U9.12 (Zd); no longer J1.28 (Pin_28), U3.21 (D7)
- net step.0: now also J1.18 (Pin_18); no longer J1.39 (Pin_39)
- net step.1: now also J1.19 (Pin_19); no longer J1.40 (Pin_40)
- net step.2: now also J1.20 (Pin_20); no longer J1.41 (Pin_41)
- net step.3: now also J1.21 (Pin_21); no longer J1.42 (Pin_42)
- new net man_ctrl: J2.26 (Pin_26), R1.1, U4.1 (S), U5.1 (S), U6.1 (S), U7.1 (S), U8.1 (S), U9.1 (S)
- new net rom1.0: U1.13 (D0), U4.2 (I0a)
- new net rom1.1: U1.14 (D1), U4.5 (I0b)
- new net rom1.2: U1.15 (D2), U4.11 (I0c)
- new net rom1.3: U1.17 (D3), U4.14 (I0d)
- new net rom1.4: U1.18 (D4), U5.2 (I0a)
- new net rom1.5: U1.19 (D5), U5.5 (I0b)
- new net rom1.6: U1.20 (D6), U5.11 (I0c)
- new net rom1.7: U1.21 (D7), U5.14 (I0d)
- new net rom2.0: U2.13 (D0), U6.2 (I0a)
- new net rom2.1: U2.14 (D1), U6.5 (I0b)
- new net rom2.2: U2.15 (D2), U6.11 (I0c)
- new net rom2.3: U2.17 (D3), U6.14 (I0d)
- new net rom2.4: U2.18 (D4), U7.2 (I0a)
- new net rom2.5: U2.19 (D5), U7.5 (I0b)
- new net rom2.6: U2.20 (D6), U7.11 (I0c)
- new net rom2.7: U2.21 (D7), U7.14 (I0d)
- new net rom3.0: U3.13 (D0), U8.2 (I0a)
- new net rom3.1: U3.14 (D1), U8.5 (I0b)
- new net rom3.2: U3.15 (D2), U8.11 (I0c)
- new net rom3.3: U3.17 (D3), U8.14 (I0d)
- new net rom3.4: U3.18 (D4), U9.2 (I0a)
- new net rom3.5: U3.19 (D5), U9.5 (I0b)
- new net rom3.6: U3.20 (D6), U9.11 (I0c)
- new net rom3.7: U3.21 (D7), U9.14 (I0d)
- new net sig1.0: J2.2 (Pin_2), RN1.1 (R1.1), U4.3 (I1a)
- new net sig1.1: J2.3 (Pin_3), RN1.2 (R2.1), U4.6 (I1b)
- new net sig1.2: J2.4 (Pin_4), RN1.3 (R3.1), U4.10 (I1c)
- new net sig1.3: J2.5 (Pin_5), RN1.4 (R4.1), U4.13 (I1d)
- new net sig1.4: J2.6 (Pin_6), RN2.1 (R1.1), U5.3 (I1a)
- new net sig1.5: J2.7 (Pin_7), RN2.2 (R2.1), U5.6 (I1b)
- new net sig1.6: J2.8 (Pin_8), RN2.3 (R3.1), U5.10 (I1c)
- new net sig1.7: J2.9 (Pin_9), RN2.4 (R4.1), U5.13 (I1d)
- new net sig2.0: J2.10 (Pin_10), RN3.1 (R1.1), U6.3 (I1a)
- new net sig2.1: J2.11 (Pin_11), RN3.2 (R2.1), U6.6 (I1b)
- new net sig2.2: J2.12 (Pin_12), RN3.3 (R3.1), U6.10 (I1c)
- new net sig2.3: J2.13 (Pin_13), RN3.4 (R4.1), U6.13 (I1d)
- new net sig2.4: J2.14 (Pin_14), RN4.1 (R1.1), U7.3 (I1a)
- new net sig2.5: J2.15 (Pin_15), RN4.2 (R2.1), U7.6 (I1b)
- new net sig2.6: J2.16 (Pin_16), RN4.3 (R3.1), U7.10 (I1c)
- new net sig2.7: J2.17 (Pin_17), RN4.4 (R4.1), U7.13 (I1d)
- new net sig3.0: J2.18 (Pin_18), RN5.1 (R1.1), U8.3 (I1a)
- new net sig3.1: J2.19 (Pin_19), RN5.2 (R2.1), U8.6 (I1b)
- new net sig3.2: J2.20 (Pin_20), RN5.3 (R3.1), U8.10 (I1c)
- new net sig3.3: J2.21 (Pin_21), RN5.4 (R4.1), U8.13 (I1d)
- new net sig3.4: J2.22 (Pin_22), RN6.1 (R1.1), U9.3 (I1a)
- new net sig3.5: J2.23 (Pin_23), RN6.2 (R2.1), U9.6 (I1b)
- new net sig3.6: J2.24 (Pin_24), RN6.3 (R3.1), U9.10 (I1c)
- new net sig3.7: J2.25 (Pin_25), RN6.4 (R4.1), U9.13 (I1d)
- no-connect marks 8 -> 6
Other:
- note added: "TESTPOINTS"
- moved on the sheet: C1, C2, C3

Commit message: CLU Controls Shield layout changes, add reg2 select switch, CLU layout changes
Parts:
- removed J2: Conn_01x28_Pin, Connector_PinSocket_2.54mm:PinSocket_1x28_P2.54mm_Vertical, symbol Connector:Conn_01x28_Pin
- added J2: Conn_01x30_Pin, Connector_PinSocket_2.54mm:PinSocket_1x30_P2.54mm_Vertical, symbol Connector:Conn_01x30_Pin
- U1, U2, U3: value SST39SF010 -> SST39SF040; symbol Memory_Flash:SST39SF010 -> Memory_Flash:SST39SF040
Connections:
- net clk is gone; now on net FETCH: J1.3 (Pin_3)
- net ~{rst} is gone; now on net EXECUTE: J1.4 (Pin_4)
- net +5V: now also J4.2 (Pin_2), J2.29 (Pin_29)
- net EXECUTE: no longer J1.6 (Pin_6)
- net FETCH: no longer J1.5 (Pin_5)
- net GND: now also U1.1 (A18), U1.30 (A17), U2.1 (A18), U2.30 (A17), U3.1 (A18), U3.30 (A17), J2.30 (Pin_30); no longer J1.46 (Pin_46), J4.2 (Pin_2)
- net INTERRUPT: now also J1.5 (Pin_5); no longer J1.7 (Pin_7)
- net aflags.cf: now also J1.13 (Pin_13); no longer J1.15 (Pin_15)
- net aflags.nf: now also J1.14 (Pin_14); no longer J1.16 (Pin_16)
- net aflags.vf: now also J1.15 (Pin_15); no longer J1.17 (Pin_17)
- net aflags.zf: now also J1.12 (Pin_12); no longer J1.14 (Pin_14)
- net man_ctrl: now also J2.28 (Pin_28)
- net opcode.0: now also J1.6 (Pin_6); no longer J1.8 (Pin_8)
- net opcode.1: now also J1.7 (Pin_7); no longer J1.9 (Pin_9)
- net opcode.2: now also J1.8 (Pin_8); no longer J1.10 (Pin_10)
- net opcode.3: now also J1.9 (Pin_9); no longer J1.11 (Pin_11)
- net opcode.4: now also J1.10 (Pin_10); no longer J1.12 (Pin_12)
- net opcode.5: now also J1.11 (Pin_11); no longer J1.13 (Pin_13)
- net q1.0: now also J1.20 (Pin_20); no longer J1.22 (Pin_22)
- net q1.1: now also J1.21 (Pin_21); no longer J1.23 (Pin_23)
- net q1.2: now also J1.22 (Pin_22); no longer J1.24 (Pin_24)
- net q1.3: now also J1.23 (Pin_23); no longer J1.25 (Pin_25)
- net q1.4: now also J1.24 (Pin_24); no longer J1.26 (Pin_26)
- net q1.5: now also J1.25 (Pin_25); no longer J1.27 (Pin_27)
- net q1.6: now also J1.26 (Pin_26); no longer J1.28 (Pin_28)
- net q1.7: now also J1.27 (Pin_27); no longer J1.29 (Pin_29)
- net q2.0: now also J1.28 (Pin_28); no longer J1.30 (Pin_30)
- net q2.1: now also J1.29 (Pin_29); no longer J1.31 (Pin_31)
- net q2.2: now also J1.30 (Pin_30); no longer J1.32 (Pin_32)
- net q2.3: now also J1.31 (Pin_31); no longer J1.33 (Pin_33)
- net q2.4: now also J1.32 (Pin_32); no longer J1.34 (Pin_34)
- net q2.5: now also J1.33 (Pin_33); no longer J1.35 (Pin_35)
- net q2.6: now also J1.34 (Pin_34); no longer J1.36 (Pin_36)
- net q2.7: now also J1.35 (Pin_35); no longer J1.37 (Pin_37)
- net q3.0: now also J1.36 (Pin_36); no longer J1.38 (Pin_38)
- net q3.1: now also J1.37 (Pin_37); no longer J1.39 (Pin_39)
- net q3.2: now also J1.38 (Pin_38); no longer J1.40 (Pin_40)
- net q3.3: now also J1.39 (Pin_39); no longer J1.41 (Pin_41)
- net q3.4: now also J1.40 (Pin_40); no longer J1.42 (Pin_42)
- net q3.5: now also J1.41 (Pin_41); no longer J1.43 (Pin_43)
- net q3.6: now also J1.42 (Pin_42); no longer J1.44 (Pin_44)
- net q3.7: now also J1.43 (Pin_43); no longer J1.45 (Pin_45)
- net sig1.0: now also J2.1 (Pin_1)
- net sig1.1: now also J2.2 (Pin_2)
- net sig1.2: now also J2.3 (Pin_3)
- net sig1.3: now also J2.4 (Pin_4)
- net sig1.4: now also J2.5 (Pin_5)
- net sig1.5: now also J2.6 (Pin_6)
- net sig1.6: now also J2.7 (Pin_7)
- net sig1.7: now also J2.8 (Pin_8)
- net sig2.0: now also J2.9 (Pin_9)
- net sig2.1: now also J2.10 (Pin_10)
- net sig2.2: now also J2.11 (Pin_11)
- net sig2.3: now also J2.12 (Pin_12)
- net sig2.4: now also J2.13 (Pin_13)
- net sig2.5: now also J2.14 (Pin_14)
- net sig2.6: now also J2.15 (Pin_15)
- net sig2.7: now also J2.16 (Pin_16)
- net sig3.0: now also J2.17 (Pin_17)
- net sig3.1: now also J2.18 (Pin_18)
- net sig3.2: now also J2.19 (Pin_19)
- net sig3.3: now also J2.20 (Pin_20)
- net sig3.4: now also J2.21 (Pin_21)
- net sig3.5: now also J2.22 (Pin_22)
- net sig3.6: now also J2.23 (Pin_23)
- net sig3.7: now also J2.24 (Pin_24)
- net step.0: now also J1.16 (Pin_16); no longer J1.18 (Pin_18)
- net step.1: now also J1.17 (Pin_17); no longer J1.19 (Pin_19)
- net step.2: now also J1.18 (Pin_18); no longer J1.20 (Pin_20)
- net step.3: now also J1.19 (Pin_19); no longer J1.21 (Pin_21)
- new net reg2_sig.0: J1.44 (Pin_44), J2.25 (Pin_25)
- new net reg2_sig.1: J1.45 (Pin_45), J2.26 (Pin_26)
- new net reg2_sig.2: J1.46 (Pin_46), J2.27 (Pin_27)
- no-connect marks 6 -> 0
Other:
- moved on the sheet: J3, J4
